Commit message: Added the nodes for dealing with 2 cameras and 2 POIs.

File: src/digital_twin/urdf/random_sphere_1.urdf.xacro (robot description, xacro)
@@ -1,7 +1,7 @@
 <?xml version="1.0" encoding="utf-8"?>
 <robot xmlns:xacro="http://www.ros.org/wiki/xacro" name="digital_twin">
-  <xacro:property name="sphere_x" value="${0.2}"/>
-  <xacro:property name="sphere_y" value="${-0.4}"/>
-  <xacro:property name="sphere_z" value="${0.2}"/>
+  <xacro:property name="red_2_sphere_x" value="${0.1}"/>
+  <xacro:property name="red_2_sphere_y" value="${-0.3}"/>
+  <xacro:property name="red_2_sphere_z" value="${0.1}"/>
   <xacro:property name="red_sphere_x" value="${0.2}"/>
   <xacro:property name="red_sphere_y" value="${-0.4}"/>
@@ -32,4 +32,28 @@
     <origin xyz="${red_sphere_x} ${red_sphere_y} ${red_sphere_z}" rpy="0 0 0"/>
    </joint>
+     <link name="red_sphere_2">
+    <inertial>
+      <mass value="0.0001"/>
+      <inertia ixx="0.0001" ixy="0" ixz="0" iyy="0.0001" iyz="0" izz="0.0001"/>
+    </inertial>
+    <visual>
+      <geometry>
+        <sphere radius="0.02"/>
+      </geometry>
+      <material name="red">
+        <color rgba="1 0 0 1"/>
+      </material>
+    </visual>
+    <collision>
+      <geometry>
+        <sphere radius="0.09"/>
+      </geometry>
+    </collision>
+  </link>
+   <joint name="joint_name_2" type="fixed">
+    <parent link="world"/>
+    <child link="red_sphere_2"/>
+    <origin xyz="${red_2_sphere_x} ${red_2_sphere_y} ${red_2_sphere_z}" rpy="0 0 0"/>
+   </joint>
 <!--
   <link name="black_sphere">
